File: kicad/esc/connectors.kicad_sch (KiCad schematic)
At the start: 0 parts

Commit message: RC1
Parts:
- added J1: ~, Connector_PinHeader_2.54mm:PinHeader_1x10_P2.54mm_Vertical, symbol ESC Custom:SignalHeader
- added J3: Screw_Terminal_01x02, TerminalBlock_4Ucon:TerminalBlock_4Ucon_1x02_P3.50mm_Vertical, symbol Connector:Screw_Terminal_01x02
Connections:
- new net +12V: J3.1 (Pin_1)
- new net GND: J3.2 (Pin_2)
- new net GND_EXT: J1.1 (EXT_GND)
- new net U_HI: J1.10 (U_HI)
- new net U_LO: J1.9 (U_LO)
- new net U_SENSE: J1.2 (U_SENSE)
- new net V_HI: J1.8 (V_HI)
- new net V_LO: J1.7 (V_LO)
- new net V_SENSE: J1.3 (V_SENSE)
- new net W_HI: J1.6 (W_HI)
- new net W_LO: J1.5 (W_LO)
- new net W_SENSE: J1.4 (W_SENSE)
